File: pcb/control-module.kicad_pcb (KiCad board)
At the start: 2 copper layers, 78.7 x 69.9 mm, 110 parts, among them J1 Screw_Terminal_01x06, J2 Conn_01x07_Pin, J3 USB_C_Receptacle_USB2.0_16P, J4 Micro_SD_Card, Q1 SiS454DN, Q2 SiS454DN, SW1 SW_DIP_x04, U1 TPS2116DRL, U2 USBLC6-2SC6, U3 STM32U545RETxQ, U4 MS5607-02BA, U5 LSM6DSL, U6 MCP73831-2-OT, U7 MIC5504-3.3YM5

Commit message: PCB Layout updates
Parts:
- moved TP_SPI_MISO1 188.6 mm to (47.2, 35.5), turned to 180 degrees
- moved TP_SPI_MOSI1 185.4 mm to (51.5, 35.5), turned to 180 degrees
- moved TP_IMU_INT1 184.1 mm to (47.5, 41.8), turned to 180 degrees
- moved TP_SPI_SCK1 181.7 mm to (57.0, 33.0), turned to 180 degrees
- moved TP_SPI_CS1 177.9 mm to (57.0, 37.2), turned to 180 degrees
- moved TP_IMU_INT2 176.8 mm to (57.0, 41.5), turned to 180 degrees
- moved BARO_CS 176.2 mm to (51.8, 57.2), turned to 90 degrees
- moved BARO_SCK 173.0 mm to (57.0, 46.2), turned to 90 degrees
- moved BARO_MOSI 171.8 mm to (57.0, 50.5), turned to 90 degrees
- moved BARO_MISO 171.1 mm to (57.0, 54.8), turned to 90 degrees
- moved P2_GNDD 161.7 mm to (136.9, -7.28)
- moved P2_OUT 155.6 mm to (142.1, 0.97)
- moved P2_FIRE 152.1 mm to (136.9, 5.22)
- moved P1_GNDD 150.8 mm to (117.7, -7.59)
- moved P2_CONT 149.6 mm to (142.1, -3.53)
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- renumbered TP_BARO_CS1 to BARO_CS, TP_BARO_MISO1 to BARO_MISO, TP_BARO_MOSI1 to BARO_MOSI, TP_BARO_SCK1 to BARO_SCK, TP_PYRO1_CONT1 to P1_CONT, TP_PYRO1_FIRE1 to P1_FIRE, TP_PYRO1_GNDD1 to P1_GNDD, TP_PYRO1_OUT1 to P1_OUT, TP_PYRO2_CONT1 to P2_CONT, TP_PYRO2_FIRE1 to P2_FIRE, TP_PYRO2_GNDD1 to P2_GNDD, TP_PYRO2_OUT1 to P2_OUT
Routing:
- net unconnected-(U3-PB0-Pad24): track 29.6 -> 0.00 mm, vias 2 -> 0
- net unconnected-(U3-PC13-Pad2): track 19.6 -> 0.00 mm, vias 2 -> 0
- net Net-(J3-CC2): track 15.2 -> 7.50 mm
- net +3.3V: track 16.6 -> 9.10 mm
- net /Pyro Controller 2/Out: track 8.48 -> 12.9 mm
- net /MCU/PYRO2_FIRE: track 12.5 -> 16.4 mm
- net /Pyro Controller 1/Out: track 9.36 -> 12.9 mm
- net /MCU/ADC1_IN5: track 20.1 -> 16.7 mm
- net /MCU/ADC1_IN6: track 16.6 -> 14.8 mm
- net Net-(Q1-G): track 1.66 -> 0.00 mm
- net /MCU/PYRO1_FIRE: track 12.1 -> 11.2 mm, vias 2 -> 0
- net /IMU Sensors/imu_int1: track 10.7 -> 9.78 mm
- net GNDD: track 32.3 -> 32.6 mm, vias 52 -> 36

Commit message: Updated PCB
Parts:
- removed TP_ADC_BAT_DIV1: TestPoint, TestPoint:TestPoint_Loop_D2.54mm_Drill1.5mm_Beaded
- moved GND_{2} 109.9 mm to (119.8, 79.0)
- moved FID1 88.6 mm to (129.2, 76.2)
- moved BARO_CS 87.1 mm to (135.0, 82.8)
- moved BARO_MISO 87.1 mm to (140.2, 80.2)
- moved BARO_MOSI 87.1 mm to (140.2, 76.0)
- moved BARO_SCK 87.1 mm to (140.2, 71.8)
- moved C15 87.1 mm to (134.8, 72.8)
- moved C16 87.1 mm to (133.2, 64.2)
- moved C17 87.1 mm to (134.8, 70.0)
- moved IMU_INT1 87.1 mm to (130.8, 67.2)
- moved IMU_INT2 87.1 mm to (140.2, 67.0)
- moved SPI_CS1 87.1 mm to (140.2, 62.8)
- moved SPI_MISO1 87.1 mm to (130.5, 61.0)
- moved SPI_MOSI1 87.1 mm to (134.8, 61.0)
- moved SPI_SCK1 87.1 mm to (140.2, 58.5)
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- renumbered TP_3V3_reg1 to 3V3_reg, TP_3V3_sd1 to 3V3_sd, TP_3V3_mcu1 to 3V3_{mcu}, TP_BATT1 to BATT, TP_BAT_SENSE_MID1 to BAT_{SENSE}, TP_BOOT1 to BOOT0, TP_GND_1 to GND_{1}, TP_GND_2 to GND_{2}, TP_IMU_INT1 to IMU_INT1, TP_IMU_INT2 to IMU_INT2, TP_Power_Mux_STAT1 to Mux_STAT, TP_NRST1 to NRST, TP_SD_CLK1 to SD_CLK, TP_SD_CMD1 to SD_CMD, TP_SD_DAT1 to SD_DAT, TP_SD_EJECT1 to SD_{EJECT}, TP_SPI_CS1 to SPI_CS1, TP_SPI_MISO1 to SPI_MISO1, TP_SPI_MOSI1 to SPI_MOSI1, TP_SPI_SCK1 to SPI_SCK1, TP_USB_D-1 to USB_D_{-}, TP_USB_D+1 to USB_{D+}, TP_V_{BAT}1 to V_{BAT}, TP_VUSB1 to V_{USB}, TP_V_USB1 to V_{USB}, TP_V_{mux}1 to V_{mux}
Routing:
- net /MCU/SD_CLK: track 10.8 -> 32.4 mm
- net /Battery/V_{mux}: track 0.00 -> 20.5 mm
- net /MCU/SD_CMD: track 11.5 -> 29.6 mm
- net /Battery/V_{BAT}: track 0.00 -> 14.3 mm
- net /MCU/SD_DAT0: track 18.7 -> 31.8 mm
- net +BATT: track 8.65 -> 21.4 mm
- net /IMU Sensors/imu_sclk: track 12.1 -> 22.7 mm
- net /Bat Sense: track 11.7 -> 20.7 mm
- net /Battery/Status: track 0.00 -> 8.72 mm
- net /IMU Sensors/imu_miso: track 6.31 -> 14.5 mm
- net /IMU Sensors/imu_cs: track 12.6 -> 19.4 mm
- net /IMU Sensors/pres_cs: track 7.33 -> 14.1 mm
- net /IMU Sensors/imu_int2: track 13.0 -> 19.8 mm
- net /IMU Sensors/imu_mosi: track 8.01 -> 14.4 mm
- net /IMU Sensors/pres_miso: track 6.36 -> 12.2 mm
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Other:
- board text added: "Battery"
- board text added: "IMU Sensors"
- board text added: "MicroSD"
- board text added: "Pyro Con. 1"
- board text added: "Pyro Con. 2"
